Commit message: updated diff bot codes

File: diff_bot/urdf/color_macros.xacro (robot description, xacro)
@@ -1,4 +1,4 @@
 <?xml version="1.0"?>
-<robot name="my_diff_bot" xmlns:xacro="http://www.ros.org/wiki/xacro" >
+<robot xmlns:xacro="http://www.ros.org/wiki/xacro" >
     <material name="white">
         <color rgba="1 1 1 1" />

File: diff_bot/urdf/controllers/emc2_hw_ros2_control.xacro (robot description, xacro)
@@ -1,10 +1,10 @@
 <?xml version="1.0"?>
-<robot name="my_diff_bot" xmlns:xacro="http://ros.org/wiki/xacro">
-    <xacro:include filename="$(find my_diff_bot)/urdf/transmission_macros.xacro"/>
-    <ros2_control name="my_diff_bot_emc2_ros2_control" type="system">
+<robot xmlns:xacro="http://ros.org/wiki/xacro">
+    <xacro:include filename="transmission_macros.xacro"/>
+    <ros2_control name="diff_bot_emc2_ros2_control" type="system">
       <hardware>
         <plugin>emc2_ros2_arduino_driver_interface/EMC2ArduinoHardware</plugin>
-        <param name="motorB_wheel_name">left_wheel_joint</param>
-        <param name="motorA_wheel_name">right_wheel_joint</param>
+        <param name="motorA_wheel_name">left_wheel_joint</param>
+        <param name="motorB_wheel_name">right_wheel_joint</param>
         <param name="port">/dev/ttyUSB0</param>
       </hardware>

File: diff_bot/urdf/controllers/transmission_macros.xacro (robot description, xacro)
@@ -1,9 +1,10 @@
 <?xml version="1.0"?>
-<robot xmlns:xacro="http://www.ros.org/wiki/xacro" name="my_diff_bot">
+<robot xmlns:xacro="http://www.ros.org/wiki/xacro">
     <xacro:macro name="insert_wheel_transmission" params="joint_name">
         <joint name="${joint_name}">
+        <!-- NOTE: velocity is in "radians/sec" and position is in "radians" -->
             <command_interface name="velocity">
-                <param name="min">-7.0</param>
-                <param name="max">7.0</param>
+                <param name="min">-7.5</param>
+                <param name="max">7.5</param>
             </command_interface>
             <state_interface name="position"/>

File: diff_bot/urdf/inertia_macros.xacro (robot description, xacro)
@@ -1,4 +1,4 @@
 <?xml version="1.0"?>
-<robot name="my_diff_bot" xmlns:xacro="http://www.ros.org/wiki/xacro" >
+<robot xmlns:xacro="http://www.ros.org/wiki/xacro" >
     <!-- Specify some standard inertial calculations https://en.wikipedia.org/wiki/List_of_moments_of_inertia -->
     <!-- These make use of xacro's mathematical functionality -->

File: diff_bot/urdf/other_parts/box_with_fillet_macro.xacro (robot description, xacro)
@@ -1,4 +1,4 @@
 <?xml version="1.0"?>
-<robot name="my_diff_bot" xmlns:xacro="http://www.ros.org/wiki/xacro" >
+<robot xmlns:xacro="http://www.ros.org/wiki/xacro" >
     <xacro:macro name="insert_box_with_fillet" params="x y z size_x size_y size_z fillet_radius material">
             <!-- logitudinal box -->
@@ -51,51 +51,3 @@
             </visual>
     </xacro:macro>
-    <xacro:macro name="insert_drive_wheel">
-        <visual>
-            <origin xyz="0 0 0" rpy="0 0 0"/>
-            <geometry>
-                <cylinder radius="0.065" length="0.06"/>
-            </geometry>
-            <material name="black"/>
-        </visual>
-        <collision>
-           <origin xyz="0 0 0" rpy="0 0 0"/>
-            <geometry>
-                <cylinder radius="0.065" length="0.06"/>
-            </geometry>
-        </collision>
-        <xacro:inertial_cylinder mass="0.2" length="0.06" radius="0.065">
-            <origin xyz="0 0 0" rpy="0 0 0"/>
-        </xacro:inertial_cylinder>
-    </xacro:macro>
-    <xacro:macro name="insert_wheel_rim">
-        <visual>
-            <origin xyz="0 0 0" rpy="0 0 0"/>
-            <geometry>
-                <box size="0.01 0.07 0.0605"/>
-            </geometry>
-            <material name="red"/>
-        </visual>
-        <visual>
-            <origin xyz="0 0 0" rpy="0 0 ${pi/2}"/>
-            <geometry>
-                <box size="0.01 0.07 0.0605"/>
-            </geometry>
-            <material name="red"/>
-        </visual>
-        <visual>
-            <origin xyz="0 0 0" rpy="0 0 ${-pi/4}"/>
-            <geometry>
-                <box size="0.01 0.07 0.0605"/>
-            </geometry>
-            <material name="red"/>
-        </visual>
-        <visual>
-            <origin xyz="0 0 0" rpy="0 0 ${pi/4}"/>
-            <geometry>
-                <box size="0.01 0.07 0.0605"/>
-            </geometry>
-            <material name="red"/>
-        </visual>
-    </xacro:macro>
 </robot>
